File: AD8232.kicad_pcb (KiCad board)
At the start: 2 copper layers, 50.1 x 45.8 mm, 33 parts, among them J1 Conn_01x03, J2 Conn_01x06, J3 AudioJack3, M1 AD8232

Commit message: agregar y ordenar silk screen del PCB
Other:
- board text added: "!SDN"
- board text added: "3.3v"
- board text added: "AD8232 Heart Monitor"
- board text added: "DO NOT USE! This is a copy of the following original board from SparkFun: https://www.sparkfun.com/products/12650"
- board text added: "Ernesto Menendez 20072392"
- board text added: "GND"
- board text added: "LA"
- board text added: "LO+"
- board text added: "LO-"
- board text added: "OUTPUT"
- board text added: "RA"
- board text added: "RL"

Commit message: definir configuracion del margen de la mascara de soldadura en PCB
Other:
- rule pad_to_mask_clearance: 0.051 -> 0.0508
- rule solder_mask_min_width: 0.25 -> 0.101
Changed lines of the file:
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@@
     (pad_size 1.524 1.524)
     (pad_drill 0.762)
-    (pad_to_mask_clearance 0.051)
-    (solder_mask_min_width 0.25)
+    (pad_to_mask_clearance 0.0508)
+    (solder_mask_min_width 0.101)
     (aux_axis_origin 0 0)
     (visible_elements FFFFFF7F)
