File: AD8232.kicad_pcb (KiCad board)
At the start: 2 copper layers, 50.1 x 45.8 mm, 33 parts, among them J1 Conn_01x03, J2 Conn_01x06, J3 AudioJack3, M1 AD8232

Commit message: corregir conexion a GND del integrado AD8232, y volver a generar los archivos gerber
Routing:
- net GND: track 18.1 -> 20.1 mm
- net +3V3: track 111.6 -> 112.1 mm
Changed lines of the file:
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@@
     (thickness 1.6)
     (drawings 29)
-    (tracks 210)
+    (tracks 213)
     (zones 0)
     (modules 33)
@@
   (segment (start 153.67 73.66) (end 156.013002 73.66) (width 0.813) (layer B.Cu) (net 9))
   (segment (start 156.013002 73.66) (end 166.173002 83.82) (width 0.813) (layer B.Cu) (net 9))
-  (segment (start 163.83 82.505) (end 163.83 82.0675) (width 0.25) (layer F.Cu) (net 9))
-  (segment (start 166.37 83.82) (end 165.145 83.82) (width 0.25) (layer F.Cu) (net 9))
-  (segment (start 165.145 83.82) (end 163.83 82.505) (width 0.25) (layer F.Cu) (net 9))
+  (segment (start 165.145 83.82) (end 163.83 82.505) (width 0.25) (layer F.Cu) (net 9) (status 1000000))
+  (segment (start 166.37 83.82) (end 165.145 83.82) (width 0.25) (layer F.Cu) (net 9) (status 1000000))
   (segment (start 168.91 85.135) (end 168.91 85.5725) (width 0.25) (layer F.Cu) (net 9))
   (segment (start 167.595 83.82) (end 168.91 85.135) (width 0.25) (layer F.Cu) (net 9))
@@
   (segment (start 164.40912 87.52732) (end 164.40912 87.90178) (width 0.25) (layer F.Cu) (net 9))
   (segment (start 166.37 83.82) (end 166.37 87.098718) (width 0.813) (layer B.Cu) (net 9))
-  (segment (start 165.7898 83.82) (end 163.05784 86.55196) (width 0.25) (layer F.Cu) (net 9))
   (segment (start 166.37 83.82) (end 165.7898 83.82) (width 0.25) (layer F.Cu) (net 9))
-  (segment (start 163.05784 86.55196) (end 163.05784 87.05088) (width 0.25) (layer F.Cu) (net 9))
   (segment (start 172.72 83.82) (end 172.72 83.82) (width 0.813) (layer B.Cu) (net 9))
   (via (at 172.72 83.82) (size 0.8) (drill 0.4) (layers F.Cu B.Cu) (net 9))
@@
   (segment (start 172.72 86.0475) (end 173.515 86.8425) (width 0.25) (layer F.Cu) (net 9))
   (segment (start 172.72 83.82) (end 172.72 86.0475) (width 0.25) (layer F.Cu) (net 9))
-  (via (at 162.56 88.9) (size 0.8) (drill 0.4) (layers F.Cu B.Cu) (net 10))
+  (segment (start 163.05784 86.55196) (end 163.05784 87.05088) (width 0.25) (layer F.Cu) (net 9))
+  (segment (start 163.05784 83.27716) (end 163.05784 86.55196) (width 0.25) (layer F.Cu) (net 9))
+  (segment (start 163.83 82.505) (end 163.05784 83.27716) (width 0.25) (layer F.Cu) (net 9))
+  (segment (start 163.83 82.0675) (end 163.83 82.505) (width 0.25) (layer F.Cu) (net 9))
   (segment (start 163.55822 87.90178) (end 163.55822 87.05088) (width 0.25) (layer F.Cu) (net 10))
   (segment (start 162.56 88.9) (end 163.55822 87.90178) (width 0.25) (layer F.Cu) (net 10))
@@
   (segment (start 171.45 78.74) (end 172.72 80.01) (width 0.25) (layer F.Cu) (net 10))
   (segment (start 169.6975 78.74) (end 169.6975 82.55) (width 0.25) (layer F.Cu) (net 10))
+  (segment (start 163.55822 87.05088) (end 163.55822 85.36178) (width 0.25) (layer F.Cu) (net 10))
+  (via (at 163.83 85.09) (size 0.8) (drill 0.4) (layers F.Cu B.Cu) (net 10))
+  (segment (start 163.55822 85.36178) (end 163.83 85.09) (width 0.25) (layer F.Cu) (net 10))
   (segment (start 165.4325 73.66) (end 162.0775 73.66) (width 0.25) (layer F.Cu) (net 11))
   (segment (start 162.0775 73.66) (end 162.0775 77.47) (width 0.25) (layer F.Cu) (net 11))
